File: hardware/gb-fpga/cartridge.sch (KiCad schematic (older format))
At the start: 5 parts, among them J2 Cartridge-32pin, U6 TXS0108E, U7 TXS0108E, U8 TXS0108E, U9 TXS0108E

Commit message: Add missing power supplies
Parts:
- added C50, C51, C52, C53, C54, C55, C56, C57: 100nF, Capacitor_SMD:C_0402_1005Metric, symbol Device:C_Small
Connections:
- net +3V3: now also C50.1, C51.1, C52.1, C53.1
- net +5V: now also C54.1, C55.1, C56.1, C57.1
- net GND: now also C50.2, C51.2, C52.2, C53.2, C54.2, C55.2, C56.2, C57.2
Other:
- moved on the sheet: J2, U6, U7, U8, U9

Commit message: Update bom
Parts:
- C50, C51, C52, C53, C54, C55, C56, C57: Manufacturer Part Number (none) -> CL05B104KO5NNNC
- U6, U7, U8, U9: Manufacturer Part Number (none) -> TXS0108EPWR
Changed lines of the file:
@@
 F 2 "Package_SO:TSSOP-20_4.4x6.5mm_P0.65mm" H 4400 1550 60  0001 L CNN
 F 3 "" H 4400 1350 60  0001 L CNN
+F 4 "TXS0108EPWR" H 4200 1500 50  0001 C CNN "Manufacturer Part Number"
 	1    4200 1500
 	1    0    0    -1
@@
 F 2 "Package_SO:TSSOP-20_4.4x6.5mm_P0.65mm" H 4400 3050 60  0001 L CNN
 F 3 "" H 4400 2850 60  0001 L CNN
+F 4 "TXS0108EPWR" H 4200 3000 50  0001 C CNN "Manufacturer Part Number"
 	1    4200 3000
 	1    0    0    -1
@@
 F 2 "Package_SO:TSSOP-20_4.4x6.5mm_P0.65mm" H 4400 4550 60  0001 L CNN
 F 3 "" H 4400 4350 60  0001 L CNN
+F 4 "TXS0108EPWR" H 4200 4500 50  0001 C CNN "Manufacturer Part Number"
 	1    4200 4500
 	1    0    0    -1
@@
 F 2 "Package_SO:TSSOP-20_4.4x6.5mm_P0.65mm" H 4400 6050 60  0001 L CNN
 F 3 "" H 4400 5850 60  0001 L CNN
+F 4 "TXS0108EPWR" H 4200 6000 50  0001 C CNN "Manufacturer Part Number"
 	1    4200 6000
 	1    0    0    -1
@@
 F 2 "Capacitor_SMD:C_0402_1005Metric" H 2500 1600 50  0001 C CNN
 F 3 "~" H 2500 1600 50  0001 C CNN
+F 4 "CL05B104KO5NNNC" H 2500 1600 50  0001 C CNN "Manufacturer Part Number"
 	1    2500 1600
 	1    0    0    -1
@@
 F 2 "Capacitor_SMD:C_0402_1005Metric" H 2500 3100 50  0001 C CNN
 F 3 "~" H 2500 3100 50  0001 C CNN
+F 4 "CL05B104KO5NNNC" H 2500 3100 50  0001 C CNN "Manufacturer Part Number"
 	1    2500 3100
 	1    0    0    -1
@@
 F 2 "Capacitor_SMD:C_0402_1005Metric" H 2500 4600 50  0001 C CNN
 F 3 "~" H 2500 4600 50  0001 C CNN
+F 4 "CL05B104KO5NNNC" H 2500 4600 50  0001 C CNN "Manufacturer Part Number"
 	1    2500 4600
 	1    0    0    -1
@@
 F 2 "Capacitor_SMD:C_0402_1005Metric" H 2500 6100 50  0001 C CNN
 F 3 "~" H 2500 6100 50  0001 C CNN
+F 4 "CL05B104KO5NNNC" H 2500 6100 50  0001 C CNN "Manufacturer Part Number"
 	1    2500 6100
 	1    0    0    -1
@@
 F 2 "Capacitor_SMD:C_0402_1005Metric" H 2950 1600 50  0001 C CNN
 F 3 "~" H 2950 1600 50  0001 C CNN
+F 4 "CL05B104KO5NNNC" H 2950 1600 50  0001 C CNN "Manufacturer Part Number"
 	1    2950 1600
 	1    0    0    -1
@@
 F 2 "Capacitor_SMD:C_0402_1005Metric" H 2950 3100 50  0001 C CNN
 F 3 "~" H 2950 3100 50  0001 C CNN
+F 4 "CL05B104KO5NNNC" H 2950 3100 50  0001 C CNN "Manufacturer Part Number"
 	1    2950 3100
 	1    0    0    -1
@@
 F 2 "Capacitor_SMD:C_0402_1005Metric" H 2950 4600 50  0001 C CNN
 F 3 "~" H 2950 4600 50  0001 C CNN
+F 4 "CL05B104KO5NNNC" H 2950 4600 50  0001 C CNN "Manufacturer Part Number"
 	1    2950 4600
 	1    0    0    -1
@@
 F 2 "Capacitor_SMD:C_0402_1005Metric" H 2950 6100 50  0001 C CNN
 F 3 "~" H 2950 6100 50  0001 C CNN
+F 4 "CL05B104KO5NNNC" H 2950 6100 50  0001 C CNN "Manufacturer Part Number"
 	1    2950 6100
 	1    0    0    -1
