File: hardware/gb-fpga/power-fpga.sch (KiCad schematic (older format))
At the start: 35 parts, among them U1 xc7s25ftgb196

Commit message: Update bom
Parts:
- C15, C19, C22, C23, C28, C29, C35, C36, C42, C43: Manufacturer Part Number (none) -> GRM035R60J475ME15D
- C16, C17, C20, C24, C25, C26, C30, C31, C32, C33, C37, C38, C39, C40, C44, C45, C46, C47: Manufacturer Part Number (none) -> GRM033R60J474KE90D
- U1: Manufacturer Part Number (none) -> XC7S25-1FTGB196C
Changed lines of the file:
@@
 F 2 "Package_BGA:Xilinx_FTGB196" H 5350 1050 60  0001 L CNN
 F 3 "" H 5350 850 60  0001 L CNN
+F 4 "XC7S25-1FTGB196C" H 5150 1000 50  0001 C CNN "Manufacturer Part Number"
 	4    5150 1000
 	1    0    0    -1
@@
 F 2 "Capacitor_SMD:C_0201_0603Metric" H 3500 5800 50  0001 C CNN
 F 3 "~" H 3500 5800 50  0001 C CNN
+F 4 "GRM033R60J474KE90D" H 3500 5800 50  0001 C CNN "Manufacturer Part Number"
 	1    3500 5800
 	1    0    0    -1
@@
 F 2 "Capacitor_SMD:C_0201_0603Metric" H 3150 5800 50  0001 C CNN
 F 3 "~" H 3150 5800 50  0001 C CNN
+F 4 "GRM035R60J475ME15D" H 3150 5800 50  0001 C CNN "Manufacturer Part Number"
 	1    3150 5800
 	1    0    0    -1
@@
 F 2 "Capacitor_SMD:C_0201_0603Metric" H 3800 5800 50  0001 C CNN
 F 3 "~" H 3800 5800 50  0001 C CNN
+F 4 "GRM033R60J474KE90D" H 3800 5800 50  0001 C CNN "Manufacturer Part Number"
 	1    3800 5800
 	1    0    0    -1
@@
 F 2 "Capacitor_SMD:C_0201_0603Metric" H 4100 5800 50  0001 C CNN
 F 3 "~" H 4100 5800 50  0001 C CNN
+F 4 "GRM033R60J474KE90D" H 4100 5800 50  0001 C CNN "Manufacturer Part Number"
 	1    4100 5800
 	1    0    0    -1
@@
 F 2 "Capacitor_SMD:C_0201_0603Metric" H 4400 5800 50  0001 C CNN
 F 3 "~" H 4400 5800 50  0001 C CNN
+F 4 "GRM033R60J474KE90D" H 4400 5800 50  0001 C CNN "Manufacturer Part Number"
 	1    4400 5800
 	1    0    0    -1
@@
 F 2 "Capacitor_SMD:C_0201_0603Metric" H 2800 5800 50  0001 C CNN
 F 3 "~" H 2800 5800 50  0001 C CNN
+F 4 "GRM035R60J475ME15D" H 2800 5800 50  0001 C CNN "Manufacturer Part Number"
 	1    2800 5800
 	1    0    0    -1
@@
 F 2 "Capacitor_SMD:C_0201_0603Metric" H 3500 5300 50  0001 C CNN
 F 3 "~" H 3500 5300 50  0001 C CNN
+F 4 "GRM033R60J474KE90D" H 3500 5300 50  0001 C CNN "Manufacturer Part Number"
 	1    3500 5300
 	1    0    0    -1
@@
 F 2 "Capacitor_SMD:C_0201_0603Metric" H 3150 5300 50  0001 C CNN
 F 3 "~" H 3150 5300 50  0001 C CNN
+F 4 "GRM035R60J475ME15D" H 3150 5300 50  0001 C CNN "Manufacturer Part Number"
 	1    3150 5300
 	1    0    0    -1
@@
 F 2 "Capacitor_SMD:C_0201_0603Metric" H 3800 5300 50  0001 C CNN
 F 3 "~" H 3800 5300 50  0001 C CNN
+F 4 "GRM033R60J474KE90D" H 3800 5300 50  0001 C CNN "Manufacturer Part Number"
 	1    3800 5300
 	1    0    0    -1
@@
 F 2 "Capacitor_SMD:C_0201_0603Metric" H 4100 5300 50  0001 C CNN
 F 3 "~" H 4100 5300 50  0001 C CNN
+F 4 "GRM033R60J474KE90D" H 4100 5300 50  0001 C CNN "Manufacturer Part Number"
 	1    4100 5300
 	1    0    0    -1
@@
 F 2 "Capacitor_SMD:C_0201_0603Metric" H 4400 5300 50  0001 C CNN
 F 3 "~" H 4400 5300 50  0001 C CNN
+F 4 "GRM033R60J474KE90D" H 4400 5300 50  0001 C CNN "Manufacturer Part Number"
 	1    4400 5300
 	1    0    0    -1
@@
 F 2 "Capacitor_SMD:C_0201_0603Metric" H 2800 5300 50  0001 C CNN
 F 3 "~" H 2800 5300 50  0001 C CNN
+F 4 "GRM035R60J475ME15D" H 2800 5300 50  0001 C CNN "Manufacturer Part Number"
 	1    2800 5300
 	1    0    0    -1
@@
 F 2 "Capacitor_SMD:C_0201_0603Metric" H 2800 4900 50  0001 C CNN
 F 3 "~" H 2800 4900 50  0001 C CNN
+F 4 "GRM035R60J475ME15D" H 2800 4900 50  0001 C CNN "Manufacturer Part Number"
 	1    2800 4900
 	1    0    0    -1
@@
 F 2 "Capacitor_SMD:C_0201_0603Metric" H 4400 4900 50  0001 C CNN
 F 3 "~" H 4400 4900 50  0001 C CNN
+F 4 "GRM033R60J474KE90D" H 4400 4900 50  0001 C CNN "Manufacturer Part Number"
 	1    4400 4900
 	1    0    0    -1
@@
 F 2 "Capacitor_SMD:C_0201_0603Metric" H 4100 4900 50  0001 C CNN
 F 3 "~" H 4100 4900 50  0001 C CNN
+F 4 "GRM033R60J474KE90D" H 4100 4900 50  0001 C CNN "Manufacturer Part Number"
 	1    4100 4900
 	1    0    0    -1
@@
 F 2 "Capacitor_SMD:C_0201_0603Metric" H 3800 4900 50  0001 C CNN
 F 3 "~" H 3800 4900 50  0001 C CNN
+F 4 "GRM033R60J474KE90D" H 3800 4900 50  0001 C CNN "Manufacturer Part Number"
 	1    3800 4900
 	1    0    0    -1
@@
 F 2 "Capacitor_SMD:C_0201_0603Metric" H 3150 4900 50  0001 C CNN
 F 3 "~" H 3150 4900 50  0001 C CNN
+F 4 "GRM035R60J475ME15D" H 3150 4900 50  0001 C CNN "Manufacturer Part Number"
 	1    3150 4900
 	1    0    0    -1
@@
 F 2 "Capacitor_SMD:C_0201_0603Metric" H 3500 4900 50  0001 C CNN
 F 3 "~" H 3500 4900 50  0001 C CNN
+F 4 "GRM033R60J474KE90D" H 3500 4900 50  0001 C CNN "Manufacturer Part Number"
 	1    3500 4900
 	1    0    0    -1
@@
 F 2 "Capacitor_SMD:C_0201_0603Metric" H 3850 3700 50  0001 C CNN
 F 3 "~" H 3850 3700 50  0001 C CNN
+F 4 "GRM033R60J474KE90D" H 3850 3700 50  0001 C CNN "Manufacturer Part Number"
 	1    3850 3700
 	1    0    0    -1
@@
 F 2 "Capacitor_SMD:C_0201_0603Metric" H 3500 3700 50  0001 C CNN
 F 3 "~" H 3500 3700 50  0001 C CNN
+F 4 "GRM035R60J475ME15D" H 3500 3700 50  0001 C CNN "Manufacturer Part Number"
 	1    3500 3700
 	1    0    0    -1
@@
 F 2 "Capacitor_SMD:C_0201_0603Metric" H 4150 3700 50  0001 C CNN
 F 3 "~" H 4150 3700 50  0001 C CNN
+F 4 "GRM033R60J474KE90D" H 4150 3700 50  0001 C CNN "Manufacturer Part Number"
 	1    4150 3700
 	1    0    0    -1
@@
 F 2 "Capacitor_SMD:C_0201_0603Metric" H 4450 3700 50  0001 C CNN
 F 3 "~" H 4450 3700 50  0001 C CNN
+F 4 "GRM033R60J474KE90D" H 4450 3700 50  0001 C CNN "Manufacturer Part Number"
 	1    4450 3700
 	1    0    0    -1
@@
 F 2 "Capacitor_SMD:C_0201_0603Metric" H 3150 3700 50  0001 C CNN
 F 3 "~" H 3150 3700 50  0001 C CNN
+F 4 "GRM035R60J475ME15D" H 3150 3700 50  0001 C CNN "Manufacturer Part Number"
 	1    3150 3700
 	1    0    0    -1
@@
 F 2 "Capacitor_SMD:C_0201_0603Metric" H 4450 3200 50  0001 C CNN
 F 3 "~" H 4450 3200 50  0001 C CNN
+F 4 "GRM033R60J474KE90D" H 4450 3200 50  0001 C CNN "Manufacturer Part Number"
 	1    4450 3200
 	1    0    0    -1
@@
 F 2 "Capacitor_SMD:C_0201_0603Metric" H 4100 3200 50  0001 C CNN
 F 3 "~" H 4100 3200 50  0001 C CNN
+F 4 "GRM035R60J475ME15D" H 4100 3200 50  0001 C CNN "Manufacturer Part Number"
 	1    4100 3200
 	1    0    0    -1
@@
 F 2 "Capacitor_SMD:C_0201_0603Metric" H 4150 2300 50  0001 C CNN
 F 3 "~" H 4150 2300 50  0001 C CNN
+F 4 "GRM033R60J474KE90D" H 4150 2300 50  0001 C CNN "Manufacturer Part Number"
 	1    4150 2300
 	1    0    0    -1
@@
 F 2 "Capacitor_SMD:C_0201_0603Metric" H 3800 2300 50  0001 C CNN
 F 3 "~" H 3800 2300 50  0001 C CNN
+F 4 "GRM035R60J475ME15D" H 3800 2300 50  0001 C CNN "Manufacturer Part Number"
 	1    3800 2300
 	1    0    0    -1
@@
 F 2 "Capacitor_SMD:C_0201_0603Metric" H 4450 2300 50  0001 C CNN
 F 3 "~" H 4450 2300 50  0001 C CNN
+F 4 "GRM033R60J474KE90D" H 4450 2300 50  0001 C CNN "Manufacturer Part Number"
 	1    4450 2300
 	1    0    0    -1

Commit message: Update footprints and BOM
Parts:
- C14, C18: footprint Capacitor_SMD:C_0201_0603Metric -> Capacitor_SMD:C_0603_1608Metric; Manufacturer Part Number (none) -> CL10A476MQ8QRNC
- C21, C27, C34, C41: footprint Capacitor_SMD:C_0201_0603Metric -> Capacitor_SMD:C_1206_3216Metric; Manufacturer Part Number (none) -> GRM31CR61A107ME05L
Changed lines of the file:
@@
 F 0 "C41" H 2500 5850 50  0000 L CNN
 F 1 "100µF" H 2500 5750 50  0000 L CNN
-F 2 "Capacitor_SMD:C_0201_0603Metric" H 2450 5800 50  0001 C CNN
+F 2 "Capacitor_SMD:C_1206_3216Metric" H 2450 5800 50  0001 C CNN
 F 3 "~" H 2450 5800 50  0001 C CNN
+F 4 "GRM31CR61A107ME05L" H 2450 5800 50  0001 C CNN "Manufacturer Part Number"
 	1    2450 5800
 	1    0    0    -1
@@
 F 0 "C34" H 2500 5350 50  0000 L CNN
 F 1 "100µF" H 2500 5250 50  0000 L CNN
-F 2 "Capacitor_SMD:C_0201_0603Metric" H 2450 5300 50  0001 C CNN
+F 2 "Capacitor_SMD:C_1206_3216Metric" H 2450 5300 50  0001 C CNN
 F 3 "~" H 2450 5300 50  0001 C CNN
+F 4 "GRM31CR61A107ME05L" H 2450 5300 50  0001 C CNN "Manufacturer Part Number"
 	1    2450 5300
 	1    0    0    -1
@@
 F 0 "C27" H 2500 4950 50  0000 L CNN
 F 1 "100µF" H 2500 4850 50  0000 L CNN
-F 2 "Capacitor_SMD:C_0201_0603Metric" H 2450 4900 50  0001 C CNN
+F 2 "Capacitor_SMD:C_1206_3216Metric" H 2450 4900 50  0001 C CNN
 F 3 "~" H 2450 4900 50  0001 C CNN
+F 4 "GRM31CR61A107ME05L" H 2450 4900 50  0001 C CNN "Manufacturer Part Number"
 	1    2450 4900
 	1    0    0    -1
@@
 F 0 "C21" H 2850 3750 50  0000 L CNN
 F 1 "100µF" H 2850 3650 50  0000 L CNN
-F 2 "Capacitor_SMD:C_0201_0603Metric" H 2800 3700 50  0001 C CNN
+F 2 "Capacitor_SMD:C_1206_3216Metric" H 2800 3700 50  0001 C CNN
 F 3 "~" H 2800 3700 50  0001 C CNN
+F 4 "GRM31CR61A107ME05L" H 2800 3700 50  0001 C CNN "Manufacturer Part Number"
 	1    2800 3700
 	1    0    0    -1
@@
 F 0 "C18" H 3800 3250 50  0000 L CNN
 F 1 "47µF" H 3800 3150 50  0000 L CNN
-F 2 "Capacitor_SMD:C_0201_0603Metric" H 3750 3200 50  0001 C CNN
+F 2 "Capacitor_SMD:C_0603_1608Metric" H 3750 3200 50  0001 C CNN
 F 3 "~" H 3750 3200 50  0001 C CNN
+F 4 "CL10A476MQ8QRNC" H 3750 3200 50  0001 C CNN "Manufacturer Part Number"
 	1    3750 3200
 	1    0    0    -1
@@
 F 0 "C14" H 3500 2350 50  0000 L CNN
 F 1 "47µF" H 3500 2250 50  0000 L CNN
-F 2 "Capacitor_SMD:C_0201_0603Metric" H 3450 2300 50  0001 C CNN
+F 2 "Capacitor_SMD:C_0603_1608Metric" H 3450 2300 50  0001 C CNN
 F 3 "~" H 3450 2300 50  0001 C CNN
+F 4 "CL10A476MQ8QRNC" H 3450 2300 50  0001 C CNN "Manufacturer Part Number"
 	1    3450 2300
 	1    0    0    -1
