File: hardware/gb-fpga/power.sch (KiCad schematic (older format))
At the start: 39 parts, among them J3 BAT+, J4 BAT-, Q1 MBT3904DW1, SW1 Switch, U4 LTC3555, U5 TLV61046ADB

Commit message: Update bom
Parts:
- C11, C5: Manufacturer Part Number (none) -> GRM155R60J226ME11D
- C12: Manufacturer Part Number (none) -> CL05A105KO5NNNC
- C13: Manufacturer Part Number (none) -> CL05A475KP5NRNC
- C3: Manufacturer Part Number (none) -> CL05A474KP5NNNC
- C4, C6, C8: Manufacturer Part Number (none) -> CL05C220JB5NNNC
- C7, C9: Manufacturer Part Number (none) -> CL05A106MP5NUNC
- D3: Manufacturer Part Number (none) -> NCD0402B1
- L1: Manufacturer Part Number (none) -> SDFL1005Q1R5KTF
- L2, L4: Manufacturer Part Number (none) -> SDFL1005Q3R3KTF
- L3: Manufacturer Part Number (none) -> SDFL1005Q2R2KTF
- Q1: Manufacturer Part Number (none) -> MBT3904DW1T1H
- R18, R27: Manufacturer Part Number (none) -> RC0402FR-073KL
- R19: Manufacturer Part Number (none) -> RC0402FR-072KL
- R20, R29, R30: Manufacturer Part Number (none) -> AF0402FR-0730KL
- R21, R23: Manufacturer Part Number (none) -> RC0402FR-07120KL
- R22: Manufacturer Part Number (none) -> RC0402FR-07150KL
- R24, R34: Manufacturer Part Number (none) -> RC0402FR-07180KL
- R25: Manufacturer Part Number (none) -> RC0402FR-0757K6L
- R26, R28: Manufacturer Part Number (none) -> RC0402JR-0710KL
- R31: Manufacturer Part Number (none) -> RC0402JR-071KL
- R32: Manufacturer Part Number (none) -> AC0402JR-07200RL
- R33: Manufacturer Part Number (none) -> RC0402FR-07953KL
- SW1: Manufacturer Part Number (none) -> EG2215
- U4: Manufacturer Part Number (none) -> LTC3555IUFD-1#PBF
- U5: Manufacturer Part Number (none) -> TLV61046ADBVR
Changed lines of the file:
@@
 F 2 "Package_DFN_QFN:QFN-28-1EP_4x5mm_P0.5mm_EP2.65x3.65mm" H 4500 3550 50  0001 C CNN
 F 3 "https://www.analog.com/media/en/technical-documentation/data-sheets/3555fe.pdf" H 4500 3550 50  0001 C CNN
+F 4 "LTC3555IUFD-1#PBF" H 4500 3600 50  0001 C CNN "Manufacturer Part Number"
 	1    4500 3600
 	1    0    0    -1
@@
 F 2 "Resistor_SMD:R_0402_1005Metric" H 3200 4550 50  0001 C CNN
 F 3 "~" H 3200 4550 50  0001 C CNN
+F 4 "RC0402FR-073KL" H 3200 4550 50  0001 C CNN "Manufacturer Part Number"
 	1    3200 4550
 	1    0    0    -1
@@
 F 2 "Capacitor_SMD:C_0402_1005Metric" H 3050 4550 50  0001 C CNN
 F 3 "~" H 3050 4550 50  0001 C CNN
+F 4 "CL05A474KP5NNNC" H 3050 4550 50  0001 C CNN "Manufacturer Part Number"
 	1    3050 4550
 	1    0    0    -1
@@
 F 2 "Resistor_SMD:R_0402_1005Metric" H 3600 4750 50  0001 C CNN
 F 3 "~" H 3600 4750 50  0001 C CNN
+F 4 "RC0402FR-072KL" H 3600 4750 50  0001 C CNN "Manufacturer Part Number"
 	1    3600 4750
 	1    0    0    -1
@@
 F 2 "Inductor_SMD:L_0402_1005Metric" H 5800 3700 50  0001 C CNN
 F 3 "~" H 5800 3700 50  0001 C CNN
+F 4 "SDFL1005Q1R5KTF" H 5800 3700 50  0001 C CNN "Manufacturer Part Number"
 	1    5800 3700
 	0    -1   -1   0
@@
 F 2 "Capacitor_SMD:C_0402_1005Metric" H 6000 3800 50  0001 C CNN
 F 3 "~" H 6000 3800 50  0001 C CNN
+F 4 "CL05C220JB5NNNC" H 6000 3800 50  0001 C CNN "Manufacturer Part Number"
 	1    6000 3800
 	1    0    0    -1
@@
 F 2 "Resistor_SMD:R_0402_1005Metric" H 6400 3800 50  0001 C CNN
 F 3 "~" H 6400 3800 50  0001 C CNN
+F 4 "AF0402FR-0730KL" H 6400 3800 50  0001 C CNN "Manufacturer Part Number"
 	1    6400 3800
 	1    0    0    -1
@@
 F 2 "Resistor_SMD:R_0402_1005Metric" H 6700 3900 50  0001 C CNN
 F 3 "~" H 6700 3900 50  0001 C CNN
+F 4 "RC0402FR-07120KL" H 6700 3900 50  0001 C CNN "Manufacturer Part Number"
 	1    6700 3900
 	0    1    1    0
@@
 F 2 "Capacitor_SMD:C_0402_1005Metric" H 6850 3800 50  0001 C CNN
 F 3 "~" H 6850 3800 50  0001 C CNN
+F 4 "GRM155R60J226ME11D" H 6850 3800 50  0001 C CNN "Manufacturer Part Number"
 	1    6850 3800
 	1    0    0    -1
@@
 F 2 "Inductor_SMD:L_0402_1005Metric" H 5800 4100 50  0001 C CNN
 F 3 "~" H 5800 4100 50  0001 C CNN
+F 4 "SDFL1005Q3R3KTF" H 5800 4100 50  0001 C CNN "Manufacturer Part Number"
 	1    5800 4100
 	0    -1   -1   0
@@
 F 2 "Capacitor_SMD:C_0402_1005Metric" H 6000 4200 50  0001 C CNN
 F 3 "~" H 6000 4200 50  0001 C CNN
+F 4 "CL05C220JB5NNNC" H 6000 4200 50  0001 C CNN "Manufacturer Part Number"
 	1    6000 4200
 	1    0    0    -1
@@
 F 2 "Resistor_SMD:R_0402_1005Metric" H 6400 4200 50  0001 C CNN
 F 3 "~" H 6400 4200 50  0001 C CNN
+F 4 "RC0402FR-07150KL" H 6400 4200 50  0001 C CNN "Manufacturer Part Number"
 	1    6400 4200
 	1    0    0    -1
@@
 F 2 "Resistor_SMD:R_0402_1005Metric" H 6700 4300 50  0001 C CNN
 F 3 "~" H 6700 4300 50  0001 C CNN
+F 4 "RC0402FR-07120KL" H 6700 4300 50  0001 C CNN "Manufacturer Part Number"
 	1    6700 4300
 	0    1    1    0
@@
 F 2 "Capacitor_SMD:C_0402_1005Metric" H 6850 4200 50  0001 C CNN
 F 3 "~" H 6850 4200 50  0001 C CNN
+F 4 "CL05A106MP5NUNC" H 6850 4200 50  0001 C CNN "Manufacturer Part Number"
 	1    6850 4200
 	1    0    0    -1
@@
 F 2 "Inductor_SMD:L_0402_1005Metric" H 5800 4500 50  0001 C CNN
 F 3 "~" H 5800 4500 50  0001 C CNN
+F 4 "SDFL1005Q2R2KTF" H 5800 4500 50  0001 C CNN "Manufacturer Part Number"
 	1    5800 4500
 	0    -1   -1   0
@@
 F 2 "Capacitor_SMD:C_0402_1005Metric" H 6000 4600 50  0001 C CNN
 F 3 "~" H 6000 4600 50  0001 C CNN
+F 4 "CL05C220JB5NNNC" H 6000 4600 50  0001 C CNN "Manufacturer Part Number"
 	1    6000 4600
 	1    0    0    -1
@@
 F 2 "Resistor_SMD:R_0402_1005Metric" H 6400 4600 50  0001 C CNN
 F 3 "~" H 6400 4600 50  0001 C CNN
+F 4 "RC0402FR-07180KL" H 6400 4600 50  0001 C CNN "Manufacturer Part Number"
 	1    6400 4600
 	1    0    0    -1
@@
 F 2 "Resistor_SMD:R_0402_1005Metric" H 6700 4700 50  0001 C CNN
 F 3 "~" H 6700 4700 50  0001 C CNN
+F 4 "RC0402FR-0757K6L" H 6700 4700 50  0001 C CNN "Manufacturer Part Number"
 	1    6700 4700
 	0    1    1    0
@@
 F 2 "Capacitor_SMD:C_0402_1005Metric" H 6850 4600 50  0001 C CNN
 F 3 "~" H 6850 4600 50  0001 C CNN
+F 4 "CL05A106MP5NUNC" H 6850 4600 50  0001 C CNN "Manufacturer Part Number"
 	1    6850 4600
 	1    0    0    -1
@@
 F 2 "Capacitor_SMD:C_0402_1005Metric" H 6500 2950 50  0001 C CNN
 F 3 "~" H 6500 2950 50  0001 C CNN
+F 4 "GRM155R60J226ME11D" H 6500 2950 50  0001 C CNN "Manufacturer Part Number"
 	1    6500 2950
 	1    0    0    -1
@@
 F 2 "Inductor_SMD:L_0402_1005Metric" H 5350 2900 50  0001 C CNN
 F 3 "~" H 5350 2900 50  0001 C CNN
+F 4 "SDFL1005Q3R3KTF" H 5350 2900 50  0001 C CNN "Manufacturer Part Number"
 	1    5350 2900
 	0    -1   -1   0
@@
 F 2 "Resistor_SMD:R_0402_1005Metric" H 1600 3700 50  0001 C CNN
 F 3 "~" H 1600 3700 50  0001 C CNN
+F 4 "RC0402JR-0710KL" H 1600 3700 50  0001 C CNN "Manufacturer Part Number"
 	1    1600 3700
 	1    0    0    -1
@@
 F 2 "Resistor_SMD:R_0402_1005Metric" H 2500 3900 50  0001 C CNN
 F 3 "~" H 2500 3900 50  0001 C CNN
+F 4 "RC0402JR-0710KL" H 2500 3900 50  0001 C CNN "Manufacturer Part Number"
 	1    2500 3900
 	1    0    0    -1
@@
 F 2 "Resistor_SMD:R_0402_1005Metric" H 2300 3800 50  0001 C CNN
 F 3 "~" H 2300 3800 50  0001 C CNN
+F 4 "RC0402FR-073KL" H 2300 3800 50  0001 C CNN "Manufacturer Part Number"
 	1    2300 3800
 	0    -1   -1   0
@@
 F 2 "Package_TO_SOT_SMD:SOT-363_SC-70-6" H 2200 4950 50  0001 C CNN
 F 3 "http://www.onsemi.com/pub_link/Collateral/MBT3904DW1T1-D.PDF" H 2000 4850 50  0001 C CNN
+F 4 "MBT3904DW1T1H" H 2000 4850 50  0001 C CNN "Manufacturer Part Number"
 	1    2000 4850
 	1    0    0    -1
@@
 F 2 "Package_TO_SOT_SMD:SOT-363_SC-70-6" H 1900 5400 50  0001 C CNN
 F 3 "http://www.onsemi.com/pub_link/Collateral/MBT3904DW1T1-D.PDF" H 1700 5300 50  0001 C CNN
+F 4 "MBT3904DW1T1H" H 1700 5300 50  0001 C CNN "Manufacturer Part Number"
 	2    1700 5300
 	1    0    0    -1
@@
 F 2 "Resistor_SMD:R_0402_1005Metric" H 1300 5300 50  0001 C CNN
 F 3 "~" H 1300 5300 50  0001 C CNN
+F 4 "RC0402JR-071KL" H 1300 5300 50  0001 C CNN "Manufacturer Part Number"
 	1    1300 5300
 	0    -1   -1   0
@@
 F 2 "Resistor_SMD:R_0402_1005Metric" H 2000 4500 50  0001 C CNN
 F 3 "~" H 2000 4500 50  0001 C CNN
+F 4 "AF0402FR-0730KL" H 2000 4500 50  0001 C CNN "Manufacturer Part Number"
 	1    2000 4500
 	0    -1   -1   0
@@
 F 2 "Resistor_SMD:R_0402_1005Metric" H 1800 4650 50  0001 C CNN
 F 3 "~" H 1800 4650 50  0001 C CNN
+F 4 "AF0402FR-0730KL" H 1800 4650 50  0001 C CNN "Manufacturer Part Number"
 	1    1800 4650
 	1    0    0    -1
@@
 F 2 "LED_SMD:LED_0402_1005Metric" V 2950 3000 50  0001 C CNN
 F 3 "~" V 2950 3000 50  0001 C CNN
+F 4 "NCD0402B1" H 2950 3000 50  0001 C CNN "Manufacturer Part Number"
 	1    2950 3000
 	0    -1   -1   0
@@
 F 2 "Resistor_SMD:R_0402_1005Metric" H 2950 2650 50  0001 C CNN
 F 3 "~" H 2950 2650 50  0001 C CNN
+F 4 "AC0402JR-07200RL" H 2950 2650 50  0001 C CNN "Manufacturer Part Number"
 	1    2950 2650
 	1    0    0    -1
@@
 F 2 "Package_TO_SOT_SMD:SOT-23-6" H 9550 3250 50  0001 L CIN
 F 3 "http://www.ti.com/lit/ds/symlink/tlv61046a.pdf" H 9500 3500 50  0001 C CNN
+F 4 "TLV61046ADBVR" H 9500 3400 50  0001 C CNN "Manufacturer Part Number"
 	1    9500 3400
 	1    0    0    -1
@@
 F 2 "Capacitor_SMD:C_0402_1005Metric" H 8750 2900 50  0001 C CNN
 F 3 "~" H 8750 2900 50  0001 C CNN
+F 4 "CL05A105KO5NNNC" H 8750 2900 50  0001 C CNN "Manufacturer Part Number"
 	1    8750 2900
 	1    0    0    -1
@@
 F 2 "Resistor_SMD:R_0402_1005Metric" H 10100 3300 50  0001 C CNN
 F 3 "~" H 10100 3300 50  0001 C CNN
+F 4 "RC0402FR-07953KL" H 10100 3300 50  0001 C CNN "Manufacturer Part Number"
 	1    10100 3300
 	1    0    0    -1
@@
 F 2 "Resistor_SMD:R_0402_1005Metric" H 10100 3600 50  0001 C CNN
 F 3 "~" H 10100 3600 50  0001 C CNN
+F 4 "RC0402FR-07180KL" H 10100 3600 50  0001 C CNN "Manufacturer Part Number"
 	1    10100 3600
 	1    0    0    -1
@@
 F 2 "Capacitor_SMD:C_0402_1005Metric" H 10550 3300 50  0001 C CNN
 F 3 "~" H 10550 3300 50  0001 C CNN
+F 4 "CL05A475KP5NRNC" H 10550 3300 50  0001 C CNN "Manufacturer Part Number"
 	1    10550 3300
 	1    0    0    -1
@@
 F 2 "gb-fpga:EG2215" H 7350 2800 50  0001 C CNN
 F 3 "" H 7350 2800 50  0001 C CNN
+F 4 "EG2215" H 7350 2800 50  0001 C CNN "Manufacturer Part Number"
 	1    7350 2800
 	1    0    0    -1

Commit message: Update footprints and BOM
Parts:
- L5: footprint Inductor_SMD:L_0402_1005Metric -> Inductor_SMD:L_0603_1608Metric; Manufacturer Part Number (none) -> SDFL1608S100KTF
Changed lines of the file:
@@
 F 0 "L5" V 9600 2850 50  0000 L CNN
 F 1 "10µH" V 9600 2550 50  0000 L CNN
-F 2 "Inductor_SMD:L_0402_1005Metric" H 9500 2800 50  0001 C CNN
+F 2 "Inductor_SMD:L_0603_1608Metric" H 9500 2800 50  0001 C CNN
 F 3 "~" H 9500 2800 50  0001 C CNN
+F 4 "SDFL1608S100KTF" H 9500 2800 50  0001 C CNN "Manufacturer Part Number"
 	1    9500 2800
 	0    -1   -1   0
