File: hardware/cpu-board/kicad/gb-fpga.kicad_pcb (KiCad board)
At the start: 4 copper layers, 80.1 x 78.6 mm, 151 parts, among them J1 USB_C_Receptacle_USB2.0, J2 Cartridge-32pin, J3 BAT+, J4 BAT-, J5 Conn_02x25_Counter_Clockwise, Q1 MBT3904DW1, SW1 Switch, U1 xc7s25ftgb196, U2 MX25R3235FZBxx1, U3 FT2232HQ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

Commit message: Clean up track and rename rev
Routing:
- net DISP_B0: track 26.6 -> 24.6 mm
Other:
- board text added: "BOARD A - REV 4"
- board text removed: "BOARD A - REV 3"
