File: hardware/hi-board/kicad/hi-board.kicad_pcb (KiCad board)
At the start: 4 copper layers, 81 x 117 mm, 68 parts, among them J1 Conn_02x25_Counter_Clockwise, J2 Speaker, SW1 Up, SW2 A, SW3 Down, SW4 B, SW5 Left, SW6 Start, SW7 Right, SW8 Select, U1 LM386, U2 ER-TFT040-2, U3 TLV61046ADB, U4 ME6216A30M3G, U5 LSF0108, U6 LSF0108, U7 LSF0108, U8 LSF0108

Commit message: Place more caps
Parts:
- added C20: 100µF, Capacitor_SMD:C_1210_3225Metric, B.Cu at (60.4, -58.7)
- moved C8 112.8 mm to (59.3, -72.0)
- moved C9 109.7 mm to (47.9, -74.5)
- moved C14 109.2 mm to (59.2, -66.6)
- moved C10 91.2 mm to (37.9, -74.6)
- moved C15 90.7 mm to (47.8, -63.6)
- moved C16 85.4 mm to (38.1, -63.5)
- moved C13 84.2 mm to (28.7, -81.3)
- moved C11 79.9 mm to (28.1, -75.3)
- moved C17 79.9 mm to (28.4, -63.0)
- moved C12 77.7 mm to (24.7, -81.3)
Changed lines of the file:
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@@
     (tracks 0)
     (zones 0)
-    (modules 68)
+    (modules 69)
     (nets 100)
   )
@@
   )
   (module Capacitor_SMD:C_0603_1608Metric (layer B.Cu)
-    (at -45.075001 -29.064999 180)
+    (at 59.27 -72.02 180)
     (descr "Capacitor SMD 0603 (1608 Metric), square (rectangular) end terminal, IPC_7351 nominal, (Body size source: IPC-SM-782 page 76, https://www.pcb-3d.com/wordpress/wp-content/uploads/ipc-sm-782a_amendment_1_and_2.pdf), generated with kicad-footprint-generator")
     (tags capacitor)
@@
   )
   (module Capacitor_SMD:C_0603_1608Metric (layer B.Cu)
-    (at -54.555001 -35.384999 180)
+    (at 47.9 -74.49 180)
     (descr "Capacitor SMD 0603 (1608 Metric), square (rectangular) end terminal, IPC_7351 nominal, (Body size source: IPC-SM-782 page 76, https://www.pcb-3d.com/wordpress/wp-content/uploads/ipc-sm-782a_amendment_1_and_2.pdf), generated with kicad-footprint-generator")
     (tags capacitor)
@@
   )
   (module Capacitor_SMD:C_0603_1608Metric (layer B.Cu)
-    (at -41.065001 -29.064999 180)
+    (at 37.94 -74.6 180)
     (descr "Capacitor SMD 0603 (1608 Metric), square (rectangular) end terminal, IPC_7351 nominal, (Body size source: IPC-SM-782 page 76, https://www.pcb-3d.com/wordpress/wp-content/uploads/ipc-sm-782a_amendment_1_and_2.pdf), generated with kicad-footprint-generator")
     (tags capacitor)
@@
   )
   (module Capacitor_SMD:C_0603_1608Metric (layer B.Cu)
-    (at -37.055001 -29.064999 180)
+    (at 28.15 -75.31 180)
     (descr "Capacitor SMD 0603 (1608 Metric), square (rectangular) end terminal, IPC_7351 nominal, (Body size source: IPC-SM-782 page 76, https://www.pcb-3d.com/wordpress/wp-content/uploads/ipc-sm-782a_amendment_1_and_2.pdf), generated with kicad-footprint-generator")
     (tags capacitor)
@@
   )
   (module Capacitor_SMD:C_0603_1608Metric (layer B.Cu)
-    (at -37.055001 -34.084999 180)
+    (at 24.73 -81.27 180)
     (descr "Capacitor SMD 0603 (1608 Metric), square (rectangular) end terminal, IPC_7351 nominal, (Body size source: IPC-SM-782 page 76, https://www.pcb-3d.com/wordpress/wp-content/uploads/ipc-sm-782a_amendment_1_and_2.pdf), generated with kicad-footprint-generator")
     (tags capacitor)
@@
   )
   (module Capacitor_SMD:C_0603_1608Metric (layer B.Cu)
-    (at -41.065001 -34.084999 180)
+    (at 28.66 -81.32 180)
     (descr "Capacitor SMD 0603 (1608 Metric), square (rectangular) end terminal, IPC_7351 nominal, (Body size source: IPC-SM-782 page 76, https://www.pcb-3d.com/wordpress/wp-content/uploads/ipc-sm-782a_amendment_1_and_2.pdf), generated with kicad-footprint-generator")
     (tags capacitor)
@@
   )
   (module Capacitor_SMD:C_0603_1608Metric (layer B.Cu)
-    (at -45.075001 -34.084999 180)
+    (at 59.18 -66.57 180)
     (descr "Capacitor SMD 0603 (1608 Metric), square (rectangular) end terminal, IPC_7351 nominal, (Body size source: IPC-SM-782 page 76, https://www.pcb-3d.com/wordpress/wp-content/uploads/ipc-sm-782a_amendment_1_and_2.pdf), generated with kicad-footprint-generator")
     (tags capacitor)
@@
   )
   (module Capacitor_SMD:C_0603_1608Metric (layer B.Cu)
-    (at -37.055001 -31.574999 180)
+    (at 47.78 -63.59 180)
     (descr "Capacitor SMD 0603 (1608 Metric), square (rectangular) end terminal, IPC_7351 nominal, (Body size source: IPC-SM-782 page 76, https://www.pcb-3d.com/wordpress/wp-content/uploads/ipc-sm-782a_amendment_1_and_2.pdf), generated with kicad-footprint-generator")
     (tags capacitor)
@@
   )
   (module Capacitor_SMD:C_0603_1608Metric (layer B.Cu)
-    (at -41.065001 -31.574999 180)
+    (at 38.15 -63.45 180)
     (descr "Capacitor SMD 0603 (1608 Metric), square (rectangular) end terminal, IPC_7351 nominal, (Body size source: IPC-SM-782 page 76, https://www.pcb-3d.com/wordpress/wp-content/uploads/ipc-sm-782a_amendment_1_and_2.pdf), generated with kicad-footprint-generator")
     (tags capacitor)
@@
   )
   (module Capacitor_SMD:C_0603_1608Metric (layer B.Cu)
-    (at -45.075001 -31.574999 180)
+    (at 28.39 -62.96 180)
     (descr "Capacitor SMD 0603 (1608 Metric), square (rectangular) end terminal, IPC_7351 nominal, (Body size source: IPC-SM-782 page 76, https://www.pcb-3d.com/wordpress/wp-content/uploads/ipc-sm-782a_amendment_1_and_2.pdf), generated with kicad-footprint-generator")
     (tags capacitor)
@@
     (model ${KISYS3DMOD}/Capacitor_SMD.3dshapes/C_1210_3225Metric.wrl
       (at (xyz 0 0 0))
+      (scale (xyz 1 1 1))
+      (rotate (xyz 0 0 0))
+    )
+  )
+  (module Capacitor_SMD:C_1210_3225Metric (layer B.Cu)
+    (at 60.41 -58.71 180)
+    (descr "Capacitor SMD 1210 (3225 Metric), square (rectangular) end terminal, IPC_7351 nominal, (Body size source: IPC-SM-782 page 76, https://www.pcb-3d.com/wordpress/wp-content/uploads/ipc-sm-782a_amendment_1_and_2.pdf), generated with kicad-footprint-generator")
+    (tags capacitor)
+    (attr smd)
+    (fp_text reference C20 (at 0 2.3) (layer B.SilkS)
+      (effects (font (size 1 1) (thickness 0.15)) (justify mirror))
+    )
+    (fp_text value 100µF (at 0 -2.3) (layer B.Fab)
+      (effects (font (size 1 1) (thickness 0.15)) (justify mirror))
+    )
+    (fp_line (start 2.3 -1.6) (end -2.3 -1.6) (layer B.CrtYd) (width 0.05))
+    (fp_line (start 2.3 1.6) (end 2.3 -1.6) (layer B.CrtYd) (width 0.05))
+    (fp_line (start -2.3 1.6) (end 2.3 1.6) (layer B.CrtYd) (width 0.05))
+    (fp_line (start -2.3 -1.6) (end -2.3 1.6) (layer B.CrtYd) (width 0.05))
+    (fp_line (start -0.711252 -1.36) (end 0.711252 -1.36) (layer B.SilkS) (width 0.12))
+    (fp_line (start -0.711252 1.36) (end 0.711252 1.36) (layer B.SilkS) (width 0.12))
+    (fp_line (start 1.6 -1.25) (end -1.6 -1.25) (layer B.Fab) (width 0.1))
+    (fp_line (start 1.6 1.25) (end 1.6 -1.25) (layer B.Fab) (width 0.1))
+    (fp_line (start -1.6 1.25) (end 1.6 1.25) (layer B.Fab) (width 0.1))
+    (fp_line (start -1.6 -1.25) (end -1.6 1.25) (layer B.Fab) (width 0.1))
+    (fp_text user %R (at 0 0) (layer B.Fab)
+      (effects (font (size 0.8 0.8) (thickness 0.12)) (justify mirror))
+    )
+    (pad 1 smd roundrect (at -1.475 0 180) (size 1.15 2.7) (layers B.Cu B.Paste B.Mask) (roundrect_rratio 0.217391)
+      (net 4 GND))
+    (pad 2 smd roundrect (at 1.475 0 180) (size 1.15 2.7) (layers B.Cu B.Paste B.Mask) (roundrect_rratio 0.217391)
+      (net 6 VOUT))
+    (model ${KISYS3DMOD}/Capacitor_SMD.3dshapes/C_1210_3225Metric.wrl
+      (at (xyz 0 0 0))

Commit message: Place remaining fix components
Parts:
- removed J1: Conn_02x25_Counter_Clockwise, Connector_FFC-FPC:Hirose_FH12-50S-0.5SH_1x50-1MP_P0.50mm_Horizontal
- removed U2: ER-TFT040-2, hi-board:HRS_FH28-60S-0.5SH(05)
- added BOARD1: Conn_02x25_Counter_Clockwise, Connector_FFC-FPC:Hirose_FH12-50S-0.5SH_1x50-1MP_P0.50mm_Horizontal, B.Cu at (40.5, -46.0)
- added DISPLAY: ER-TFT040-2, hi-board:HRS_FH28-60S-0.5SH(05), B.Cu at (40.5, -82.0)
- moved RV1 55.0 mm to (7.10, -80.5), turned to 270 degrees
- moved C11 4.09 mm to (28.3, -71.2)
- moved C15 4.09 mm to (48.0, -59.5)
- moved C16 4.09 mm to (38.3, -59.4)
- moved C17 4.09 mm to (28.6, -58.9)
- moved C20 4.09 mm to (60.6, -54.6)
- moved U5 4.09 mm to (53.0, -65.3)
- moved U6 4.09 mm to (43.1, -65.2)
- moved U7 4.09 mm to (34.0, -65.2)
- moved U8 4.09 mm to (24.6, -65.3)
- moved C14 4.09 mm to (59.4, -62.5)
- moved C10 4.09 mm to (38.1, -70.5)
- moved C12 4.09 mm to (24.9, -77.2)
- moved C13 4.09 mm to (28.8, -77.2)
- moved C8 4.09 mm to (59.5, -67.9)
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