File: hardware/hi-board/kicad/hi-board.sch (KiCad schematic (older format))
At the start: 0 parts

Commit message: Add testpoints
Changed lines of the file:
@@
 $Descr A4 11693 8268
 encoding utf-8
-Sheet 1 6
+Sheet 1 7
 Title "FPGAMB0 (HI Board)"
 Date ""
@@
 F1 "joypad.sch" 50
 $EndSheet
+$Sheet
+S 2050 4400 500  150
+U 6167F82D
+F0 "Testpoints" 50
+F1 "testpoints.sch" 50
+$EndSheet
 $EndSCHEMATC
