File: hardware/hi-board/kicad/joypad.sch (KiCad schematic (older format))
At the start: 16 parts, among them SW1 Up, SW2 A, SW3 Down, SW4 B, SW5 Left, SW6 Start, SW7 Right, SW8 Select

Commit message: Add joypad footprints
Parts:
- SW1, SW2, SW3, SW4, SW5, SW7: footprint (none) -> hi-board:Rubber_Round
- SW6, SW8: footprint (none) -> hi-board:Rubber_Square
Changed lines of the file:
@@
 F 0 "SW1" H 4200 3035 50  0000 C CNN
 F 1 "Up" H 4200 2944 50  0000 C CNN
-F 2 "" H 4200 2950 50  0001 C CNN
+F 2 "hi-board:Rubber_Round" H 4200 2950 50  0001 C CNN
 F 3 "~" H 4200 2950 50  0001 C CNN
 	1    4200 2750
@@
 F 0 "SW3" H 4200 3835 50  0000 C CNN
 F 1 "Down" H 4200 3744 50  0000 C CNN
-F 2 "" H 4200 3750 50  0001 C CNN
+F 2 "hi-board:Rubber_Round" H 4200 3750 50  0001 C CNN
 F 3 "~" H 4200 3750 50  0001 C CNN
 	1    4200 3550
@@
 F 0 "SW5" H 4200 4635 50  0000 C CNN
 F 1 "Left" H 4200 4544 50  0000 C CNN
-F 2 "" H 4200 4550 50  0001 C CNN
+F 2 "hi-board:Rubber_Round" H 4200 4550 50  0001 C CNN
 F 3 "~" H 4200 4550 50  0001 C CNN
 	1    4200 4350
@@
 F 0 "SW7" H 4200 5435 50  0000 C CNN
 F 1 "Right" H 4200 5344 50  0000 C CNN
-F 2 "" H 4200 5350 50  0001 C CNN
+F 2 "hi-board:Rubber_Round" H 4200 5350 50  0001 C CNN
 F 3 "~" H 4200 5350 50  0001 C CNN
 	1    4200 5150
@@
 F 0 "SW2" H 6300 3035 50  0000 C CNN
 F 1 "A" H 6300 2944 50  0000 C CNN
-F 2 "" H 6300 2950 50  0001 C CNN
+F 2 "hi-board:Rubber_Round" H 6300 2950 50  0001 C CNN
 F 3 "~" H 6300 2950 50  0001 C CNN
 	1    6300 2750
@@
 F 0 "SW4" H 6300 3835 50  0000 C CNN
 F 1 "B" H 6300 3744 50  0000 C CNN
-F 2 "" H 6300 3750 50  0001 C CNN
+F 2 "hi-board:Rubber_Round" H 6300 3750 50  0001 C CNN
 F 3 "~" H 6300 3750 50  0001 C CNN
 	1    6300 3550
@@
 F 0 "SW6" H 6300 4635 50  0000 C CNN
 F 1 "Start" H 6300 4544 50  0000 C CNN
-F 2 "" H 6300 4550 50  0001 C CNN
+F 2 "hi-board:Rubber_Square" H 6300 4550 50  0001 C CNN
 F 3 "~" H 6300 4550 50  0001 C CNN
 	1    6300 4350
@@
 F 0 "SW8" H 6300 5435 50  0000 C CNN
 F 1 "Select" H 6300 5344 50  0000 C CNN
-F 2 "" H 6300 5350 50  0001 C CNN
+F 2 "hi-board:Rubber_Square" H 6300 5350 50  0001 C CNN
 F 3 "~" H 6300 5350 50  0001 C CNN
 	1    6300 5150

Commit message: Complete display schematic and change footprints
Parts:
- R10, R11, R12, R13, R14, R15, R16, R9: footprint Resistor_SMD:R_0402_1005Metric -> Resistor_SMD:R_0603_1608Metric
Changed lines of the file:
@@
 F 0 "R9" H 4659 2646 50  0000 L CNN
 F 1 "10k" H 4659 2555 50  0000 L CNN
-F 2 "Resistor_SMD:R_0402_1005Metric" H 4600 2600 50  0001 C CNN
+F 2 "Resistor_SMD:R_0603_1608Metric" H 4600 2600 50  0001 C CNN
 F 3 "~" H 4600 2600 50  0001 C CNN
 	1    4600 2600
@@
 F 0 "R11" H 4659 3446 50  0000 L CNN
 F 1 "10k" H 4659 3355 50  0000 L CNN
-F 2 "Resistor_SMD:R_0402_1005Metric" H 4600 3400 50  0001 C CNN
+F 2 "Resistor_SMD:R_0603_1608Metric" H 4600 3400 50  0001 C CNN
 F 3 "~" H 4600 3400 50  0001 C CNN
 	1    4600 3400
@@
 F 0 "R13" H 4659 4246 50  0000 L CNN
 F 1 "10k" H 4659 4155 50  0000 L CNN
-F 2 "Resistor_SMD:R_0402_1005Metric" H 4600 4200 50  0001 C CNN
+F 2 "Resistor_SMD:R_0603_1608Metric" H 4600 4200 50  0001 C CNN
 F 3 "~" H 4600 4200 50  0001 C CNN
 	1    4600 4200
@@
 F 0 "R15" H 4659 5046 50  0000 L CNN
 F 1 "10k" H 4659 4955 50  0000 L CNN
-F 2 "Resistor_SMD:R_0402_1005Metric" H 4600 5000 50  0001 C CNN
+F 2 "Resistor_SMD:R_0603_1608Metric" H 4600 5000 50  0001 C CNN
 F 3 "~" H 4600 5000 50  0001 C CNN
 	1    4600 5000
@@
 F 0 "R10" H 6759 2646 50  0000 L CNN
 F 1 "10k" H 6759 2555 50  0000 L CNN
-F 2 "Resistor_SMD:R_0402_1005Metric" H 6700 2600 50  0001 C CNN
+F 2 "Resistor_SMD:R_0603_1608Metric" H 6700 2600 50  0001 C CNN
 F 3 "~" H 6700 2600 50  0001 C CNN
 	1    6700 2600
@@
 F 0 "R12" H 6759 3446 50  0000 L CNN
 F 1 "10k" H 6759 3355 50  0000 L CNN
-F 2 "Resistor_SMD:R_0402_1005Metric" H 6700 3400 50  0001 C CNN
+F 2 "Resistor_SMD:R_0603_1608Metric" H 6700 3400 50  0001 C CNN
 F 3 "~" H 6700 3400 50  0001 C CNN
 	1    6700 3400
@@
 F 0 "R14" H 6759 4246 50  0000 L CNN
 F 1 "10k" H 6759 4155 50  0000 L CNN
-F 2 "Resistor_SMD:R_0402_1005Metric" H 6700 4200 50  0001 C CNN
+F 2 "Resistor_SMD:R_0603_1608Metric" H 6700 4200 50  0001 C CNN
 F 3 "~" H 6700 4200 50  0001 C CNN
 	1    6700 4200
@@
 F 0 "R16" H 6759 5046 50  0000 L CNN
 F 1 "10k" H 6759 4955 50  0000 L CNN
-F 2 "Resistor_SMD:R_0402_1005Metric" H 6700 5000 50  0001 C CNN
+F 2 "Resistor_SMD:R_0603_1608Metric" H 6700 5000 50  0001 C CNN
 F 3 "~" H 6700 5000 50  0001 C CNN
 	1    6700 5000
